Commit message: fix camera position in go2

File: resources/robots/go2/urdf/go2.urdf (robot description, URDF)
Before this commit: robot go2_description, 29 links, 28 joints
Links:
- link FL_calf: geometry collision cylinder length=0.12 radius=0.012; visual mesh filename=../meshes/calf.dae
- link FL_foot: geometry collision sphere radius=0.022; visual mesh filename=../meshes/foot.dae
- link FL_hip: geometry collision cylinder length=0.04 radius=0.046; visual mesh filename=../meshes/hip.dae
- link FL_thigh: geometry collision box size=0.213 0.0245 0.034; visual mesh filename=../meshes/thigh.dae
- link FR_calf: geometry collision cylinder length=0.12 radius=0.013; visual mesh filename=../meshes/calf_mirror.dae
- link FR_foot: geometry collision sphere radius=0.022; visual mesh filename=../meshes/foot.dae
- link FR_hip: geometry collision cylinder length=0.04 radius=0.046; visual mesh filename=../meshes/hip.dae
- link FR_thigh: geometry collision box size=0.213 0.0245 0.034; visual mesh filename=../meshes/thigh_mirror.dae
- link RL_calf: geometry collision cylinder length=0.12 radius=0.013; visual mesh filename=../meshes/calf.dae
- link RL_foot: geometry collision sphere radius=0.022; visual mesh filename=../meshes/foot.dae
- link RL_hip: geometry collision cylinder length=0.04 radius=0.046; visual mesh filename=../meshes/hip.dae
- link RL_thigh: geometry collision box size=0.213 0.0245 0.034; visual mesh filename=../meshes/thigh.dae
- link RR_calf: geometry collision cylinder length=0.12 radius=0.013; visual mesh filename=../meshes/calf_mirror.dae
- link RR_foot: geometry collision sphere radius=0.022; visual mesh filename=../meshes/foot.dae
- link RR_hip: geometry collision cylinder length=0.04 radius=0.046; visual mesh filename=../meshes/hip.dae
- link RR_thigh: geometry collision box size=0.213 0.0245 0.034; visual mesh filename=../meshes/thigh_mirror.dae
- link base: geometry collision box size=0.3762 0.0935 0.114; visual mesh filename=../meshes/trunk.dae
