Commit message: Add UniLab-style G1 foot sole capsules for fuller ground contact.
Co-authored-by: Cursor <cursoragent@cursor.com>

File: resources/robots/g1/g1_12dof.urdf (robot description, URDF)
Before this commit: robot g1_12dof, 31 links, 30 joints
Links:
- link left_ankle_roll_link: geometry collision cylinder length=0.05 radius=0.01; collision cylinder length=0.05 radius=0.01
- link right_ankle_roll_link: geometry collision cylinder length=0.05 radius=0.01; collision cylinder length=0.05 radius=0.01
